File: DND_Tower.kicad_pcb (KiCad board)
At the start: 2 copper layers, 24 x 24 mm, 17 parts, among them J1 +, J2 +, U1 ATtiny1616-M

Commit message: add git hash placeholder
Other:
- board text added: "<<hash>>"
